File: MRCS-Candlestick-Mic.brd (EAGLE design)
At the start: 54.6 x 54.6 mm, 4 parts

Commit message: silkscreen cleanup, pad update
Parts:
- moved U$3 8.89 mm to (38.1, 25.4)
Other:
- board text added: "+ RED"
- board text removed: "RED +"
